File: TH-555-VCO/mainboard-kicad/mainboard.kicad_pcb (KiCad board)
At the start: 2 copper layers, 108 x 48.3 mm, 75 parts, among them IC1 555N, IC2 LM13700N, IC3 TL074P, IC4 TL074P, T3 -NPN-TO92-EBC, T4 -PNP-TO92-EBC, T5 -PNP-TO92-EBC

Commit message: Align footprints to actual shapes
Parts:
- removed @HOLE0, @HOLE1, @HOLE2, @HOLE3: , 
- IC3, IC4: footprint Package_SO:SOIC-14_3.9x8.7mm_P1.27mm -> Package_SO:SO-14_3.9x8.65mm_P1.27mm
