File: TH-555-VCO/mainboard-kicad/mainboard.kicad_sch (KiCad schematic)
At the start: 71 parts, among them IC1 555N, IC2 LM13700N, IC3 TL074P, IC4 TL074P, T3 -NPN-TO92-EBC, T4 -PNP-TO92-EBC, T5 -PNP-TO92-EBC

Commit message: Kicost experiment: Add a few manufacturer codes
Unfortunately, many of the LCSC parts aren't picked up with these
codes. So we'll so the merged BOM manually for now.
Parts:
- C1: mpn (none) -> CC1H103ZA1FD3F4D1001
- C11: mpn (none) -> UPW2A100MED
- C13: mpn (none) -> CC1H102MA1EDB44B1100
- C3: mpn (none) -> CC1H104ZA1ED3F5O1100
- C4: mpn (none) -> H471K050BN48230L502
- C5: mpn (none) -> CC1H101KC1EDSL4B1100
- C6: mpn (none) -> Y5V222M1KV16CC0035
- IC1: mpn (none) -> NE555N
- IC2: mpn (none) -> LM13700M
- IC3: mpn (none) -> TL074CDR
- R11: mpn (none) -> 3296W-1-104
- R18: mpn (none) -> 3296W-1-101
- R40: mpn (none) -> 3296W-1-253
- T3: mpn (none) -> 2N3904
- T4: mpn (none) -> 2N3906
Changed lines of the file:
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@@
+      (effects (font (size 1.27 1.27)) hide)
+    )
+    (property "mpn" "CC1H102MA1EDB44B1100" (id 4) (at 152.4 149.86 0)
       (effects (font (size 1.27 1.27)) hide)
     )
@@
     )
     (property "Datasheet" "" (id 3) (at 398.78 219.71 0)
+      (effects (font (size 1.27 1.27)) hide)
+    )
+    (property "mpn" "LM13700M" (id 4) (at 106.68 46.99 0)
       (effects (font (size 1.27 1.27)) hide)
     )
@@
       (effects (font (size 1.27 1.27)) hide)
     )
+    (property "mpn" "NE555N" (id 4) (at 172.72 152.4 0)
+      (effects (font (size 1.27 1.27)) hide)
+    )
     (pin "1")
     (pin "2")
@@
     )
     (property "Datasheet" "" (id 3) (at 93.98 220.98 0)
+      (effects (font (size 1.27 1.27)) hide)
+    )
+    (property "mpn" "H471K050BN48230L502" (id 4) (at 93.98 220.98 0)
       (effects (font (size 1.27 1.27)) hide)
     )
@@
       (effects (font (size 1.27 1.27)) hide)
     )
+    (property "mpn" "TL074CDR" (id 4) (at 153.67 49.53 0)
+      (effects (font (size 1.27 1.27)) hide)
+    )
     (pin "1")
     (pin "2")
@@
     )
     (property "Datasheet" "" (id 3) (at 314.96 81.28 0)
+      (effects (font (size 1.27 1.27)) hide)
+    )
+    (property "mpn" "LM13700M" (id 4) (at 106.68 46.99 0)
       (effects (font (size 1.27 1.27)) hide)
     )
@@
       (effects (font (size 1.27 1.27)) hide)
     )
+    (property "mpn" "CC1H103ZA1FD3F4D1001" (id 4) (at 330.835 205.74 0)
+      (effects (font (size 1.27 1.27)) hide)
+    )
     (pin "1")
     (pin "2")
@@
       (effects (font (size 1.27 1.27)) hide)
     )
+    (property "mpn" "3296W-1-101" (id 4) (at 99.06 116.84 90)
+      (effects (font (size 1.27 1.27)) hide)
+    )
     (pin "A")
     (pin "E")
@@
     )
     (property "Datasheet" "" (id 3) (at 351.79 81.28 0)
+      (effects (font (size 1.27 1.27)) hide)
+    )
+    (property "mpn" "LM13700M" (id 4) (at 106.68 46.99 0)
       (effects (font (size 1.27 1.27)) hide)
     )
@@
       (effects (font (size 1.27 1.27)) hide)
     )
+    (property "mpn" "TL074CDR" (id 4) (at 153.67 49.53 0)
+      (effects (font (size 1.27 1.27)) hide)
+    )
     (pin "1")
     (pin "2")
@@
       (effects (font (size 1.27 1.27)) hide)
     )
+    (property "mpn" "TL074CDR" (id 4) (at 153.67 49.53 0)
+      (effects (font (size 1.27 1.27)) hide)
+    )
     (pin "1")
     (pin "2")
@@
     )
     (property "Datasheet" "" (id 3) (at 106.68 46.99 0)
+      (effects (font (size 1.27 1.27)) hide)
+    )
+    (property "mpn" "LM13700M" (id 4) (at 106.68 46.99 0)
       (effects (font (size 1.27 1.27)) hide)
     )
@@
       (effects (font (size 1.27 1.27)) hide)
     )
+    (property "mpn" "TL074CDR" (id 4) (at 153.67 49.53 0)
+      (effects (font (size 1.27 1.27)) hide)
+    )
     (pin "1")
     (pin "2")
@@
       (effects (font (size 1.27 1.27)) hide)
     )
+    (property "mpn" "UPW2A100MED" (id 4) (at 320.675 203.2 0)
+      (effects (font (size 1.27 1.27)) hide)
+    )
     (pin "+")
     (pin "-")
@@
       (effects (font (size 1.27 1.27)) hide)
     )
+    (property "mpn" "3296W-1-253" (id 4) (at 327.66 111.76 90)
+      (effects (font (size 1.27 1.27)) hide)
+    )
     (pin "A")
     (pin "E")
@@
       (effects (font (size 1.27 1.27)) hide)
     )
+    (property "mpn" "CC1H101KC1EDSL4B1100" (id 4) (at 86.36 180.34 0)
+      (effects (font (size 1.27 1.27)) hide)
+    )
     (pin "1")
     (pin "2")
@@
       (effects (font (size 1.27 1.27)) hide)
     )
+    (property "mpn" "Y5V222M1KV16CC0035" (id 4) (at 129.54 54.61 0)
+      (effects (font (size 1.27 1.27)) hide)
+    )
     (pin "1")
     (pin "2")
@@
     )
     (property "Datasheet" "" (id 3) (at 172.72 127 0)
+      (effects (font (size 1.27 1.27)) hide)
+    )
+    (property "mpn" "CC1H104ZA1ED3F5O1100" (id 4) (at 172.72 127 0)
       (effects (font (size 1.27 1.27)) hide)
     )
@@
     )
     (property "Datasheet" "" (id 3) (at 139.7 220.98 0)
+      (effects (font (size 1.27 1.27)) hide)
+    )
+    (property "mpn" "2N3904" (id 4) (at 139.7 220.98 0)
       (effects (font (size 1.27 1.27)) hide)
     )
@@
       (effects (font (size 1.27 1.27)) hide)
     )
+    (property "mpn" "TL074CDR" (id 4) (at 153.67 49.53 0)
+      (effects (font (size 1.27 1.27)) hide)
+    )
     (pin "1")
     (pin "2")
@@
       (effects (font (size 1.27 1.27)) hide)
     )
+    (property "mpn" "2N3906" (id 4) (at 88.9 160.02 0)
+      (effects (font (size 1.27 1.27)) hide)
+    )
     (pin "B")
     (pin "C")
@@
       (effects (font (size 1.27 1.27)) hide)
     )
+    (property "mpn" "3296W-1-104" (id 4) (at 177.8 187.96 90)
+      (effects (font (size 1.27 1.27)) hide)
+    )

Commit message: Align footprints to actual shapes
Parts:
- IC2: footprint Package_SO:SO-16_5.3x10.2mm_P1.27mm -> Package_SO:SOIC-16_3.9x9.9mm_P1.27mm
- IC3, IC4: footprint Package_SO:SO-14_5.3x10.2mm_P1.27mm -> Package_SO:SO-14_3.9x8.65mm_P1.27mm
Changed lines of the file:
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@@
       (effects (font (size 1.778 1.5113)) (justify left bottom) hide)
     )
-    (property "Footprint" "Package_SO:SO-16_5.3x10.2mm_P1.27mm" (id 2) (at 398.78 219.71 0)
+    (property "Footprint" "Package_SO:SOIC-16_3.9x9.9mm_P1.27mm" (id 2) (at 398.78 219.71 0)
       (effects (font (size 1.27 1.27)) hide)
     )
@@
       (effects (font (size 1.778 1.5113)) (justify left bottom) hide)
     )
-    (property "Footprint" "Package_SO:SO-14_5.3x10.2mm_P1.27mm" (id 2) (at 187.96 223.52 0)
+    (property "Footprint" "Package_SO:SO-14_3.9x8.65mm_P1.27mm" (id 2) (at 187.96 223.52 0)
       (effects (font (size 1.27 1.27)) hide)
     )
@@
       (effects (font (size 1.778 1.5113)) (justify left bottom) hide)
     )
-    (property "Footprint" "Package_SO:SO-14_5.3x10.2mm_P1.27mm" (id 2) (at 215.9 157.48 0)
+    (property "Footprint" "Package_SO:SO-14_3.9x8.65mm_P1.27mm" (id 2) (at 215.9 157.48 0)
       (effects (font (size 1.27 1.27)) hide)
     )
@@
       (effects (font (size 1.778 1.5113)) (justify left bottom) hide)
     )
-    (property "Footprint" "Package_SO:SO-14_5.3x10.2mm_P1.27mm" (id 2) (at 275.59 115.57 0)
+    (property "Footprint" "Package_SO:SO-14_3.9x8.65mm_P1.27mm" (id 2) (at 275.59 115.57 0)
       (effects (font (size 1.27 1.27)) hide)
     )
@@
       (effects (font (size 1.778 1.5113)) (justify left bottom) hide)
     )
-    (property "Footprint" "Package_SO:SO-16_5.3x10.2mm_P1.27mm" (id 2) (at 314.96 81.28 0)
+    (property "Footprint" "Package_SO:SOIC-16_3.9x9.9mm_P1.27mm" (id 2) (at 314.96 81.28 0)
       (effects (font (size 1.27 1.27)) hide)
     )
@@
       (effects (font (size 1.778 1.5113)) (justify left bottom) hide)
     )
-    (property "Footprint" "Package_SO:SO-16_5.3x10.2mm_P1.27mm" (id 2) (at 351.79 81.28 0)
+    (property "Footprint" "Package_SO:SOIC-16_3.9x9.9mm_P1.27mm" (id 2) (at 351.79 81.28 0)
       (effects (font (size 1.27 1.27)) hide)
     )
@@
       (effects (font (size 1.778 1.5113)) (justify left bottom) hide)
     )
-    (property "Footprint" "Package_SO:SO-14_5.3x10.2mm_P1.27mm" (id 2) (at 370.205 211.455 0)
+    (property "Footprint" "Package_SO:SO-14_3.9x8.65mm_P1.27mm" (id 2) (at 370.205 211.455 0)
       (effects (font (size 1.27 1.27)) hide)
     )
@@
       (effects (font (size 1.778 1.5113)) (justify left bottom) hide)
     )
-    (property "Footprint" "Package_SO:SO-14_5.3x10.2mm_P1.27mm" (id 2) (at 200.66 52.07 0)
+    (property "Footprint" "Package_SO:SO-14_3.9x8.65mm_P1.27mm" (id 2) (at 200.66 52.07 0)
       (effects (font (size 1.27 1.27)) hide)
     )
@@
       (effects (font (size 1.778 1.5113)) (justify left bottom) hide)
     )
-    (property "Footprint" "Package_SO:SO-14_5.3x10.2mm_P1.27mm" (id 2) (at 88.9 106.68 0)
+    (property "Footprint" "Package_SO:SO-14_3.9x8.65mm_P1.27mm" (id 2) (at 88.9 106.68 0)
       (effects (font (size 1.27 1.27)) hide)
     )
@@
       (effects (font (size 1.778 1.5113)) (justify left bottom) hide)
     )
-    (property "Footprint" "Package_SO:SO-14_5.3x10.2mm_P1.27mm" (id 2) (at 153.67 49.53 0)
+    (property "Footprint" "Package_SO:SO-14_3.9x8.65mm_P1.27mm" (id 2) (at 153.67 49.53 0)
       (effects (font (size 1.27 1.27)) hide)
     )
@@
       (effects (font (size 1.778 1.5113)) (justify left bottom) hide)
     )
-    (property "Footprint" "Package_SO:SO-16_5.3x10.2mm_P1.27mm" (id 2) (at 106.68 46.99 0)
+    (property "Footprint" "Package_SO:SOIC-16_3.9x9.9mm_P1.27mm" (id 2) (at 106.68 46.99 0)
       (effects (font (size 1.27 1.27)) hide)
     )
@@
       (effects (font (size 1.778 1.5113)) (justify left bottom) hide)
     )
-    (property "Footprint" "Package_SO:SO-14_5.3x10.2mm_P1.27mm" (id 2) (at 381 211.455 0)
+    (property "Footprint" "Package_SO:SO-14_3.9x8.65mm_P1.27mm" (id 2) (at 381 211.455 0)
       (effects (font (size 1.27 1.27)) hide)
     )
@@
       (effects (font (size 1.778 1.5113)) (justify left bottom) hide)
     )
-    (property "Footprint" "Package_SO:SO-14_5.3x10.2mm_P1.27mm" (id 2) (at 246.38 118.11 0)
+    (property "Footprint" "Package_SO:SO-14_3.9x8.65mm_P1.27mm" (id 2) (at 246.38 118.11 0)
       (effects (font (size 1.27 1.27)) hide)
     )
@@
       (effects (font (size 1.778 1.5113)) (justify left bottom) hide)
     )
-    (property "Footprint" "Package_SO:SO-14_5.3x10.2mm_P1.27mm" (id 2) (at 88.9 193.04 0)
+    (property "Footprint" "Package_SO:SO-14_3.9x8.65mm_P1.27mm" (id 2) (at 88.9 193.04 0)
       (effects (font (size 1.27 1.27)) hide)
     )
@@
     )
     (path "/83d29412-3f29-4c82-a40e-04f8a4ba77e1"
-      (reference "IC2") (unit 1) (value "LM13700N") (footprint "Package_SO:SO-16_5.3x10.2mm_P1.27mm")
+      (reference "IC2") (unit 1) (value "LM13700N") (footprint "Package_SO:SOIC-16_3.9x9.9mm_P1.27mm")
     )
     (path "/3193153e-7748-4a43-abff-e008ed29b4e4"
-      (reference "IC2") (unit 2) (value "LM13700N") (footprint "Package_SO:SO-16_5.3x10.2mm_P1.27mm")
+      (reference "IC2") (unit 2) (value "LM13700N") (footprint "Package_SO:SOIC-16_3.9x9.9mm_P1.27mm")
     )
     (path "/580b3386-f608-45e3-af89-3cac7209ec17"
-      (reference "IC2") (unit 4) (value "LM13700N") (footprint "Package_SO:SO-16_5.3x10.2mm_P1.27mm")
+      (reference "IC2") (unit 4) (value "LM13700N") (footprint "Package_SO:SOIC-16_3.9x9.9mm_P1.27mm")
     )
     (path "/071a40ce-02f4-4320-adaf-134c1c6f6436"
-      (reference "IC2") (unit 5) (value "LM13700N") (footprint "Package_SO:SO-16_5.3x10.2mm_P1.27mm")
+      (reference "IC2") (unit 5) (value "LM13700N") (footprint "Package_SO:SOIC-16_3.9x9.9mm_P1.27mm")
     )
     (path "/7091f7ce-253d-4648-b58a-ed0c6668379c"
-      (reference "IC3") (unit 1) (value "TL074P") (footprint "Package_SO:SO-14_5.3x10.2mm_P1.27mm")
+      (reference "IC3") (unit 1) (value "TL074P") (footprint "Package_SO:SO-14_3.9x8.65mm_P1.27mm")
     )
     (path "/e087df3c-01b8-44c5-9c81-761ed80a0c1f"
-      (reference "IC3") (unit 2) (value "TL074P") (footprint "Package_SO:SO-14_5.3x10.2mm_P1.27mm")
+      (reference "IC3") (unit 2) (value "TL074P") (footprint "Package_SO:SO-14_3.9x8.65mm_P1.27mm")
     )
     (path "/81a74df4-3f15-475e-bb4f-9ffd21bc8c44"
-      (reference "IC3") (unit 3) (value "TL074P") (footprint "Package_SO:SO-14_5.3x10.2mm_P1.27mm")
+      (reference "IC3") (unit 3) (value "TL074P") (footprint "Package_SO:SO-14_3.9x8.65mm_P1.27mm")
     )
     (path "/295ce1a6-32b0-4c33-a786-798c6381e055"
-      (reference "IC3") (unit 4) (value "TL074P") (footprint "Package_SO:SO-14_5.3x10.2mm_P1.27mm")
+      (reference "IC3") (unit 4) (value "TL074P") (footprint "Package_SO:SO-14_3.9x8.65mm_P1.27mm")
     )
     (path "/8e51e8a3-e433-4bb5-9e46-983f1197fe54"
-      (reference "IC3") (unit 5) (value "TL074P") (footprint "Package_SO:SO-14_5.3x10.2mm_P1.27mm")
+      (reference "IC3") (unit 5) (value "TL074P") (footprint "Package_SO:SO-14_3.9x8.65mm_P1.27mm")
     )
     (path "/1f7a877d-6f7a-4a79-a109-8e2f6d4b30a9"
-      (reference "IC4") (unit 1) (value "TL074P") (footprint "Package_SO:SO-14_5.3x10.2mm_P1.27mm")
+      (reference "IC4") (unit 1) (value "TL074P") (footprint "Package_SO:SO-14_3.9x8.65mm_P1.27mm")
     )
     (path "/0bdfce04-8627-4f08-a28e-787af3e6a883"
-      (reference "IC4") (unit 2) (value "TL074P") (footprint "Package_SO:SO-14_5.3x10.2mm_P1.27mm")
+      (reference "IC4") (unit 2) (value "TL074P") (footprint "Package_SO:SO-14_3.9x8.65mm_P1.27mm")
     )
     (path "/ddf729ce-b750-4d9a-b981-e3e506cf2485"
-      (reference "IC4") (unit 3) (value "TL074P") (footprint "Package_SO:SO-14_5.3x10.2mm_P1.27mm")
+      (reference "IC4") (unit 3) (value "TL074P") (footprint "Package_SO:SO-14_3.9x8.65mm_P1.27mm")
     )
     (path "/704cdedd-a6d2-40b4-a004-7d0a503b8d02"
-      (reference "IC4") (unit 4) (value "TL074P") (footprint "Package_SO:SO-14_5.3x10.2mm_P1.27mm")
+      (reference "IC4") (unit 4) (value "TL074P") (footprint "Package_SO:SO-14_3.9x8.65mm_P1.27mm")
     )
     (path "/67d03486-aeb3-4bf5-99a3-a2302333b714"
-      (reference "IC4") (unit 5) (value "TL074P") (footprint "Package_SO:SO-14_5.3x10.2mm_P1.27mm")
+      (reference "IC4") (unit 5) (value "TL074P") (footprint "Package_SO:SO-14_3.9x8.65mm_P1.27mm")
     )
     (path "/f40dea20-76a3-45a3-ad8b-e998092e55a9"
