File: RayWilson-Dual-VCA/ioboard/ioboard.kicad_sch (KiCad schematic)
At the start: 79 parts, among them IC1 TL074P, IC2 LM13700N, Q1 2N3904, Q2 2N3906, Q3 2N3904, Q4 2N3906

Commit message: Change LM13700 to be SMD since that's the only part available
In both TME and LCSC.
Parts:
- IC2: footprint ioboard:DIL16 -> Package_SO:SO-16_5.3x10.2mm_P1.27mm
Changed lines of the file:
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@@
       (effects (font (size 1.778 1.5113)) (justify left bottom) hide)
     )
-    (property "Footprint" "ioboard:DIL16" (id 2) (at 252.73 144.78 0)
+    (property "Footprint" "Package_SO:SO-16_5.3x10.2mm_P1.27mm" (id 2) (at 252.73 144.78 0)
       (effects (font (size 1.27 1.27)) hide)
     )
@@
       (effects (font (size 1.778 1.5113)) (justify left bottom) hide)
     )
-    (property "Footprint" "ioboard:DIL16" (id 2) (at 124.46 265.43 0)
+    (property "Footprint" "Package_SO:SO-16_5.3x10.2mm_P1.27mm" (id 2) (at 124.46 265.43 0)
       (effects (font (size 1.27 1.27)) hide)
     )
@@
       (effects (font (size 1.778 1.5113)) (justify left bottom) hide)
     )
-    (property "Footprint" "ioboard:DIL16" (id 2) (at 367.03 142.24 0)
+    (property "Footprint" "Package_SO:SO-16_5.3x10.2mm_P1.27mm" (id 2) (at 367.03 142.24 0)
       (effects (font (size 1.27 1.27)) hide)
     )
@@
       (effects (font (size 1.778 1.5113)) (justify left bottom) hide)
     )
-    (property "Footprint" "ioboard:DIL16" (id 2) (at 401.32 142.24 0)
+    (property "Footprint" "Package_SO:SO-16_5.3x10.2mm_P1.27mm" (id 2) (at 401.32 142.24 0)
       (effects (font (size 1.27 1.27)) hide)
     )
@@
       (effects (font (size 1.778 1.5113)) (justify left bottom) hide)
     )
-    (property "Footprint" "ioboard:DIL16" (id 2) (at 287.02 144.78 0)
+    (property "Footprint" "Package_SO:SO-16_5.3x10.2mm_P1.27mm" (id 2) (at 287.02 144.78 0)
       (effects (font (size 1.27 1.27)) hide)
     )
@@
     )
     (path "/111067b6-9b28-4712-a854-65f9ce651e98"
-      (reference "IC2") (unit 1) (value "LM13700N") (footprint "ioboard:DIL16")
+      (reference "IC2") (unit 1) (value "LM13700N") (footprint "Package_SO:SO-16_5.3x10.2mm_P1.27mm")
     )
     (path "/39437b9f-67fe-4c4f-bd11-abf9b4b690e4"
-      (reference "IC2") (unit 2) (value "LM13700N") (footprint "ioboard:DIL16")
+      (reference "IC2") (unit 2) (value "LM13700N") (footprint "Package_SO:SO-16_5.3x10.2mm_P1.27mm")
     )
     (path "/4a937f98-856b-4aa1-a5eb-b817f07413d7"
-      (reference "IC2") (unit 3) (value "LM13700N") (footprint "ioboard:DIL16")
+      (reference "IC2") (unit 3) (value "LM13700N") (footprint "Package_SO:SO-16_5.3x10.2mm_P1.27mm")
     )
     (path "/4479ebbc-132b-49d6-89d5-11c9cddf7929"
-      (reference "IC2") (unit 4) (value "LM13700N") (footprint "ioboard:DIL16")
+      (reference "IC2") (unit 4) (value "LM13700N") (footprint "Package_SO:SO-16_5.3x10.2mm_P1.27mm")
     )
     (path "/279c7d5e-a2a5-463c-9a5f-466442a96f2a"
-      (reference "IC2") (unit 5) (value "LM13700N") (footprint "ioboard:DIL16")
+      (reference "IC2") (unit 5) (value "LM13700N") (footprint "Package_SO:SO-16_5.3x10.2mm_P1.27mm")
     )
     (path "/47de7e50-8323-450b-8255-418e128952b5"

Commit message: Replace TL047P with SMD
Since that's the only package available from LCSC.
Parts:
- IC1: footprint ioboard:DIL14 -> Package_SO:SO-14_5.3x10.2mm_P1.27mm
Changed lines of the file:
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@@
       (effects (font (size 1.778 1.5113)) (justify left bottom) hide)
     )
-    (property "Footprint" "ioboard:DIL14" (id 2) (at 231.14 99.06 0)
+    (property "Footprint" "Package_SO:SO-14_5.3x10.2mm_P1.27mm" (id 2) (at 231.14 99.06 0)
       (effects (font (size 1.27 1.27)) hide)
     )
@@
       (effects (font (size 1.778 1.5113)) (justify left bottom) hide)
     )
-    (property "Footprint" "ioboard:DIL14" (id 2) (at 345.44 97.79 0)
+    (property "Footprint" "Package_SO:SO-14_5.3x10.2mm_P1.27mm" (id 2) (at 345.44 97.79 0)
       (effects (font (size 1.27 1.27)) hide)
     )
@@
       (effects (font (size 1.778 1.5113)) (justify left bottom) hide)
     )
-    (property "Footprint" "ioboard:DIL14" (id 2) (at 386.08 55.88 0)
+    (property "Footprint" "Package_SO:SO-14_5.3x10.2mm_P1.27mm" (id 2) (at 386.08 55.88 0)
       (effects (font (size 1.27 1.27)) hide)
     )
@@
       (effects (font (size 1.778 1.5113)) (justify left bottom) hide)
     )
-    (property "Footprint" "ioboard:DIL14" (id 2) (at 95.25 259.08 0)
+    (property "Footprint" "Package_SO:SO-14_5.3x10.2mm_P1.27mm" (id 2) (at 95.25 259.08 0)
       (effects (font (size 1.27 1.27)) hide)
     )
@@
       (effects (font (size 1.778 1.5113)) (justify left bottom) hide)
     )
-    (property "Footprint" "ioboard:DIL14" (id 2) (at 271.78 57.15 0)
+    (property "Footprint" "Package_SO:SO-14_5.3x10.2mm_P1.27mm" (id 2) (at 271.78 57.15 0)
       (effects (font (size 1.27 1.27)) hide)
     )
@@
     )
     (path "/492bad17-9f5d-444a-b84e-f00693f82ba7"
-      (reference "IC1") (unit 1) (value "TL074P") (footprint "ioboard:DIL14")
+      (reference "IC1") (unit 1) (value "TL074P") (footprint "Package_SO:SO-14_5.3x10.2mm_P1.27mm")
     )
     (path "/c11567b0-0b88-44a9-8994-658b3057c42c"
-      (reference "IC1") (unit 2) (value "TL074P") (footprint "ioboard:DIL14")
+      (reference "IC1") (unit 2) (value "TL074P") (footprint "Package_SO:SO-14_5.3x10.2mm_P1.27mm")
     )
     (path "/a7e88a52-a004-4c1a-842f-ef0f86a7796b"
-      (reference "IC1") (unit 3) (value "TL074P") (footprint "ioboard:DIL14")
+      (reference "IC1") (unit 3) (value "TL074P") (footprint "Package_SO:SO-14_5.3x10.2mm_P1.27mm")
     )
     (path "/9febf117-6c13-4e66-8dd3-7b8744d37e4f"
-      (reference "IC1") (unit 4) (value "TL074P") (footprint "ioboard:DIL14")
+      (reference "IC1") (unit 4) (value "TL074P") (footprint "Package_SO:SO-14_5.3x10.2mm_P1.27mm")
     )
     (path "/aaec6a5a-1f1d-491a-a01d-2167a5533dd1"
-      (reference "IC1") (unit 5) (value "TL074P") (footprint "ioboard:DIL14")
+      (reference "IC1") (unit 5) (value "TL074P") (footprint "Package_SO:SO-14_5.3x10.2mm_P1.27mm")
     )
     (path "/111067b6-9b28-4712-a854-65f9ce651e98"

Commit message: Align potentiometer packages to standard 3-pin 0.1"
Parts:
- R1, R2, R3, R4: footprint ioboard:S64YW -> Potentiometer_THT:Potentiometer_Bourns_3296W_Vertical; symbol ioboard-eagle-import:TRIM_1234-S64YW -> Device:R_Potentiometer_Trim
Connections:
- net +12V: now also R1.1, R2.1; no longer R1.E, R2.E
- net -12V: now also R1.3, R2.3; no longer R1.A, R2.A
- net at IC2.3 (+IN), R8.2: now also R3.1, R3.2; no longer R3.E, R3.S
- net at IC2.14 (+IN), R28.2: now also R4.1, R4.2; no longer R4.E, R4.S
- net at R5.1: now also R1.2; no longer R1.S
- net at R6.1: now also R2.2; no longer R2.S
- net at R27.2: now also R4.3; no longer R4.A
- net at R7.2: now also R3.3; no longer R3.A
Changed lines of the file:
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@@
     (stroke (width 0) (type default) (color 0 0 0 0))
   )
-  (wire (pts (xy 342.9 140.97) (xy 341.63 140.97))
+  (wire (pts (xy 340.36 140.97) (xy 342.9 140.97))
     (stroke (width 0) (type default) (color 0 0 0 0))
   )
@@
     (stroke (width 0) (type default) (color 0 0 0 0))
   )
-  (wire (pts (xy 227.33 138.43) (xy 227.33 135.89))
+  (wire (pts (xy 227.33 135.89) (xy 227.33 139.7))
     (stroke (width 0) (type default) (color 0 0 0 0))
   )
@@
     (stroke (width 0) (type default) (color 0 0 0 0))
   )
-  (wire (pts (xy 237.49 166.37) (xy 237.49 168.91))
+  (wire (pts (xy 237.49 166.37) (xy 237.49 170.18))
     (stroke (width 0) (type default) (color 0 0 0 0))
   )
@@
     (stroke (width 0) (type default) (color 0 0 0 0))
   )
-  (wire (pts (xy 336.55 135.89) (xy 336.55 133.35))
+  (wire (pts (xy 336.55 133.35) (xy 336.55 137.16))
     (stroke (width 0) (type default) (color 0 0 0 0))
   )
@@
     (stroke (width 0) (type default) (color 0 0 0 0))
   )
-  (wire (pts (xy 251.46 173.99) (xy 242.57 173.99))
+  (wire (pts (xy 241.3 173.99) (xy 251.46 173.99))
     (stroke (width 0) (type default) (color 0 0 0 0))
   )
@@
     (stroke (width 0) (type default) (color 0 0 0 0))
   )
-  (wire (pts (xy 233.68 143.51) (xy 232.41 143.51))
+  (wire (pts (xy 231.14 143.51) (xy 233.68 143.51))
     (stroke (width 0) (type default) (color 0 0 0 0))
   )
@@
     (stroke (width 0) (type default) (color 0 0 0 0))
   )
-  (wire (pts (xy 336.55 148.59) (xy 336.55 146.05))
+  (wire (pts (xy 336.55 144.78) (xy 336.55 148.59))
     (stroke (width 0) (type default) (color 0 0 0 0))
   )
@@
     (stroke (width 0) (type default) (color 0 0 0 0))
   )
-  (wire (pts (xy 237.49 181.61) (xy 237.49 179.07))
+  (wire (pts (xy 237.49 177.8) (xy 237.49 181.61))
     (stroke (width 0) (type default) (color 0 0 0 0))
   )
@@
     (stroke (width 0) (type default) (color 0 0 0 0))
   )
-  (wire (pts (xy 365.76 171.45) (xy 356.87 171.45))
+  (wire (pts (xy 355.6 171.45) (xy 365.76 171.45))
     (stroke (width 0) (type default) (color 0 0 0 0))
   )
@@
     (stroke (width 0) (type default) (color 0 0 0 0))
   )
-  (wire (pts (xy 351.79 163.83) (xy 351.79 166.37))
+  (wire (pts (xy 351.79 163.83) (xy 351.79 167.64))
     (stroke (width 0) (type default) (color 0 0 0 0))
   )
@@
     (stroke (width 0) (type default) (color 0 0 0 0))
   )
-  (wire (pts (xy 227.33 151.13) (xy 227.33 148.59))
+  (wire (pts (xy 227.33 147.32) (xy 227.33 151.13))
     (stroke (width 0) (type default) (color 0 0 0 0))
   )
@@
     (stroke (width 0) (type default) (color 0 0 0 0))
   )
-  (wire (pts (xy 351.79 179.07) (xy 351.79 176.53))
+  (wire (pts (xy 351.79 175.26) (xy 351.79 179.07))
     (stroke (width 0) (type default) (color 0 0 0 0))
   )
@@
     (pin "6")
   )
-  (symbol (lib_id "ioboard-eagle-import:TRIM_1234-S64YW") (at 351.79 171.45 0) (unit 1)
+  (symbol (lib_id "Device:R_Potentiometer_Trim") (at 351.79 171.45 0) (unit 1)
     (in_bom yes) (on_board yes)
     (property "Reference" "R1" (id 0) (at 345.821 175.26 90)
@@
       (effects (font (size 1.778 1.5113)) (justify left bottom))
     )
-    (property "Footprint" "ioboard:S64YW" (id 2) (at 351.79 171.45 0)
+    (property "Footprint" "Potentiometer_THT:Potentiometer_Bourns_3296W_Vertical" (id 2) (at 351.79 171.45 0)
       (effects (font (size 1.27 1.27)) hide)
     )
-    (property "Datasheet" "" (id 3) (at 351.79 171.45 0)
+    (property "Datasheet" "~" (id 3) (at 351.79 171.45 0)
       (effects (font (size 1.27 1.27)) hide)
     )
-    (pin "A")
-    (pin "E")
-    (pin "S")
-    (pin "S@1")
+    (pin "1")
+    (pin "2")
+    (pin "3")
   )
   (symbol (lib_id "ioboard-eagle-import:ML10") (at 63.5 256.54 180) (unit 1)
@@
     (pin "2")
   )
-  (symbol (lib_id "ioboard-eagle-import:TRIM_1234-S64YW") (at 336.55 140.97 0) (unit 1)
+  (symbol (lib_id "Device:R_Potentiometer_Trim") (at 336.55 140.97 0) (unit 1)
     (in_bom yes) (on_board yes)
     (property "Reference" "R4" (id 0) (at 330.581 144.78 90)
@@
       (effects (font (size 1.778 1.5113)) (justify left bottom))
     )
-    (property "Footprint" "ioboard:S64YW" (id 2) (at 336.55 140.97 0)
+    (property "Footprint" "Potentiometer_THT:Potentiometer_Bourns_3296W_Vertical" (id 2) (at 336.55 140.97 0)
       (effects (font (size 1.27 1.27)) hide)
     )
-    (property "Datasheet" "" (id 3) (at 336.55 140.97 0)
+    (property "Datasheet" "~" (id 3) (at 336.55 140.97 0)
       (effects (font (size 1.27 1.27)) hide)
     )
-    (pin "A")
-    (pin "E")
-    (pin "S")
-    (pin "S@1")
+    (pin "1")
+    (pin "2")
+    (pin "3")
   )
   (symbol (lib_id "ioboard-eagle-import:GND") (at 63.5 281.94 0) (unit 1)
@@
     (pin "1")
   )
-  (symbol (lib_id "ioboard-eagle-import:TRIM_1234-S64YW") (at 227.33 143.51 0) (unit 1)
+  (symbol (lib_id "Device:R_Potentiometer_Trim") (at 227.33 143.51 0) (unit 1)
     (in_bom yes) (on_board yes)
     (property "Reference" "R3" (id 0) (at 221.361 147.32 90)
@@
       (effects (font (size 1.778 1.5113)) (justify left bottom))
     )
-    (property "Footprint" "ioboard:S64YW" (id 2) (at 227.33 143.51 0)
+    (property "Footprint" "Potentiometer_THT:Potentiometer_Bourns_3296W_Vertical" (id 2) (at 227.33 143.51 0)
       (effects (font (size 1.27 1.27)) hide)
     )
-    (property "Datasheet" "" (id 3) (at 227.33 143.51 0)
+    (property "Datasheet" "~" (id 3) (at 227.33 143.51 0)
       (effects (font (size 1.27 1.27)) hide)
     )
-    (pin "A")
-    (pin "E")
-    (pin "S")
-    (pin "S@1")
+    (pin "1")
+    (pin "2")
+    (pin "3")
   )
   (symbol (lib_id "ioboard-eagle-import:GND") (at 73.66 152.4 0) (unit 1)
@@
     (pin "1")
   )
-  (symbol (lib_id "ioboard-eagle-import:TRIM_1234-S64YW") (at 237.49 173.99 0) (unit 1)
+  (symbol (lib_id "Device:R_Potentiometer_Trim") (at 237.49 173.99 0) (unit 1)
     (in_bom yes) (on_board yes)
     (property "Reference" "R2" (id 0) (at 231.521 177.8 90)
@@
       (effects (font (size 1.778 1.5113)) (justify left bottom))
     )
-    (property "Footprint" "ioboard:S64YW" (id 2) (at 237.49 173.99 0)
+    (property "Footprint" "Potentiometer_THT:Potentiometer_Bourns_3296W_Vertical" (id 2) (at 237.49 173.99 0)
       (effects (font (size 1.27 1.27)) hide)
     )
-    (property "Datasheet" "" (id 3) (at 237.49 173.99 0)
+    (property "Datasheet" "~" (id 3) (at 237.49 173.99 0)
       (effects (font (size 1.27 1.27)) hide)
     )
-    (pin "A")
-    (pin "E")
-    (pin "S")
-    (pin "S@1")
+    (pin "1")
+    (pin "2")
+    (pin "3")
   )
   (symbol (lib_id "ioboard-eagle-import:R-US_0204{slash}7") (at 251.46 54.61 0) (unit 1)
@@
     )
     (path "/4bffe2c9-1997-4611-9155-60bac1583bde"
-      (reference "R1") (unit 1) (value "100k") (footprint "ioboard:S64YW")
+      (reference "R1") (unit 1) (value "100k") (footprint "Potentiometer_THT:Potentiometer_Bourns_3296W_Vertical")
     )
     (path "/b321737f-b212-4a2e-b93c-d04f90d66f02"
-      (reference "R2") (unit 1) (value "100k") (footprint "ioboard:S64YW")
+      (reference "R2") (unit 1) (value "100k") (footprint "Potentiometer_THT:Potentiometer_Bourns_3296W_Vertical")
     )
     (path "/7852383d-c5a1-49f8-b4f7-ef7bd86ea3cf"
-      (reference "R3") (unit 1) (value "2k") (footprint "ioboard:S64YW")
+      (reference "R3") (unit 1) (value "2k") (footprint "Potentiometer_THT:Potentiometer_Bourns_3296W_Vertical")
     )
     (path "/65eb661e-d895-483c-bba6-18b32f6b56be"
-      (reference "R4") (unit 1) (value "2k") (footprint "ioboard:S64YW")
+      (reference "R4") (unit 1) (value "2k") (footprint "Potentiometer_THT:Potentiometer_Bourns_3296W_Vertical")
     )
     (path "/f4b7b161-cda6-4410-927d-10a6e07c2386"

Commit message: Align footprints to actual shapes
Parts:
- IC1: footprint Package_SO:SO-14_5.3x10.2mm_P1.27mm -> Package_SO:SO-14_3.9x8.65mm_P1.27mm
- IC2: footprint Package_SO:SO-16_5.3x10.2mm_P1.27mm -> Package_SO:SOIC-16_3.9x9.9mm_P1.27mm
Changed lines of the file:
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@@
       (effects (font (size 1.778 1.5113)) (justify left bottom) hide)
     )
-    (property "Footprint" "Package_SO:SO-16_5.3x10.2mm_P1.27mm" (id 2) (at 252.73 144.78 0)
+    (property "Footprint" "Package_SO:SOIC-16_3.9x9.9mm_P1.27mm" (id 2) (at 252.73 144.78 0)
       (effects (font (size 1.27 1.27)) hide)
     )
@@
       (effects (font (size 1.778 1.5113)) (justify left bottom) hide)
     )
-    (property "Footprint" "Package_SO:SO-16_5.3x10.2mm_P1.27mm" (id 2) (at 124.46 265.43 0)
+    (property "Footprint" "Package_SO:SOIC-16_3.9x9.9mm_P1.27mm" (id 2) (at 124.46 265.43 0)
       (effects (font (size 1.27 1.27)) hide)
     )
@@
       (effects (font (size 1.778 1.5113)) (justify left bottom) hide)
     )
-    (property "Footprint" "Package_SO:SO-16_5.3x10.2mm_P1.27mm" (id 2) (at 367.03 142.24 0)
+    (property "Footprint" "Package_SO:SOIC-16_3.9x9.9mm_P1.27mm" (id 2) (at 367.03 142.24 0)
       (effects (font (size 1.27 1.27)) hide)
     )
@@
       (effects (font (size 1.778 1.5113)) (justify left bottom) hide)
     )
-    (property "Footprint" "Package_SO:SO-16_5.3x10.2mm_P1.27mm" (id 2) (at 401.32 142.24 0)
+    (property "Footprint" "Package_SO:SOIC-16_3.9x9.9mm_P1.27mm" (id 2) (at 401.32 142.24 0)
       (effects (font (size 1.27 1.27)) hide)
     )
@@
       (effects (font (size 1.778 1.5113)) (justify left bottom) hide)
     )
-    (property "Footprint" "Package_SO:SO-14_5.3x10.2mm_P1.27mm" (id 2) (at 231.14 99.06 0)
+    (property "Footprint" "Package_SO:SO-14_3.9x8.65mm_P1.27mm" (id 2) (at 231.14 99.06 0)
       (effects (font (size 1.27 1.27)) hide)
     )
@@
       (effects (font (size 1.778 1.5113)) (justify left bottom) hide)
     )
-    (property "Footprint" "Package_SO:SO-16_5.3x10.2mm_P1.27mm" (id 2) (at 287.02 144.78 0)
+    (property "Footprint" "Package_SO:SOIC-16_3.9x9.9mm_P1.27mm" (id 2) (at 287.02 144.78 0)
       (effects (font (size 1.27 1.27)) hide)
     )
@@
       (effects (font (size 1.778 1.5113)) (justify left bottom) hide)
     )
-    (property "Footprint" "Package_SO:SO-14_5.3x10.2mm_P1.27mm" (id 2) (at 345.44 97.79 0)
+    (property "Footprint" "Package_SO:SO-14_3.9x8.65mm_P1.27mm" (id 2) (at 345.44 97.79 0)
       (effects (font (size 1.27 1.27)) hide)
     )
@@
       (effects (font (size 1.778 1.5113)) (justify left bottom) hide)
     )
-    (property "Footprint" "Package_SO:SO-14_5.3x10.2mm_P1.27mm" (id 2) (at 386.08 55.88 0)
+    (property "Footprint" "Package_SO:SO-14_3.9x8.65mm_P1.27mm" (id 2) (at 386.08 55.88 0)
       (effects (font (size 1.27 1.27)) hide)
     )
@@
       (effects (font (size 1.778 1.5113)) (justify left bottom) hide)
     )
-    (property "Footprint" "Package_SO:SO-14_5.3x10.2mm_P1.27mm" (id 2) (at 95.25 259.08 0)
+    (property "Footprint" "Package_SO:SO-14_3.9x8.65mm_P1.27mm" (id 2) (at 95.25 259.08 0)
       (effects (font (size 1.27 1.27)) hide)
     )
@@
       (effects (font (size 1.778 1.5113)) (justify left bottom) hide)
     )
-    (property "Footprint" "Package_SO:SO-14_5.3x10.2mm_P1.27mm" (id 2) (at 271.78 57.15 0)
+    (property "Footprint" "Package_SO:SO-14_3.9x8.65mm_P1.27mm" (id 2) (at 271.78 57.15 0)
       (effects (font (size 1.27 1.27)) hide)
     )
@@
     )
     (path "/492bad17-9f5d-444a-b84e-f00693f82ba7"
-      (reference "IC1") (unit 1) (value "TL074P") (footprint "Package_SO:SO-14_5.3x10.2mm_P1.27mm")
+      (reference "IC1") (unit 1) (value "TL074P") (footprint "Package_SO:SO-14_3.9x8.65mm_P1.27mm")
     )
     (path "/c11567b0-0b88-44a9-8994-658b3057c42c"
-      (reference "IC1") (unit 2) (value "TL074P") (footprint "Package_SO:SO-14_5.3x10.2mm_P1.27mm")
+      (reference "IC1") (unit 2) (value "TL074P") (footprint "Package_SO:SO-14_3.9x8.65mm_P1.27mm")
     )
     (path "/a7e88a52-a004-4c1a-842f-ef0f86a7796b"
-      (reference "IC1") (unit 3) (value "TL074P") (footprint "Package_SO:SO-14_5.3x10.2mm_P1.27mm")
+      (reference "IC1") (unit 3) (value "TL074P") (footprint "Package_SO:SO-14_3.9x8.65mm_P1.27mm")
     )
     (path "/9febf117-6c13-4e66-8dd3-7b8744d37e4f"
-      (reference "IC1") (unit 4) (value "TL074P") (footprint "Package_SO:SO-14_5.3x10.2mm_P1.27mm")
+      (reference "IC1") (unit 4) (value "TL074P") (footprint "Package_SO:SO-14_3.9x8.65mm_P1.27mm")
     )
     (path "/aaec6a5a-1f1d-491a-a01d-2167a5533dd1"
-      (reference "IC1") (unit 5) (value "TL074P") (footprint "Package_SO:SO-14_5.3x10.2mm_P1.27mm")
+      (reference "IC1") (unit 5) (value "TL074P") (footprint "Package_SO:SO-14_3.9x8.65mm_P1.27mm")
     )
     (path "/111067b6-9b28-4712-a854-65f9ce651e98"
-      (reference "IC2") (unit 1) (value "LM13700N") (footprint "Package_SO:SO-16_5.3x10.2mm_P1.27mm")
+      (reference "IC2") (unit 1) (value "LM13700N") (footprint "Package_SO:SOIC-16_3.9x9.9mm_P1.27mm")
     )
     (path "/39437b9f-67fe-4c4f-bd11-abf9b4b690e4"
-      (reference "IC2") (unit 2) (value "LM13700N") (footprint "Package_SO:SO-16_5.3x10.2mm_P1.27mm")
+      (reference "IC2") (unit 2) (value "LM13700N") (footprint "Package_SO:SOIC-16_3.9x9.9mm_P1.27mm")
     )
     (path "/4a937f98-856b-4aa1-a5eb-b817f07413d7"
-      (reference "IC2") (unit 3) (value "LM13700N") (footprint "Package_SO:SO-16_5.3x10.2mm_P1.27mm")
+      (reference "IC2") (unit 3) (value "LM13700N") (footprint "Package_SO:SOIC-16_3.9x9.9mm_P1.27mm")
     )
     (path "/4479ebbc-132b-49d6-89d5-11c9cddf7929"
-      (reference "IC2") (unit 4) (value "LM13700N") (footprint "Package_SO:SO-16_5.3x10.2mm_P1.27mm")
+      (reference "IC2") (unit 4) (value "LM13700N") (footprint "Package_SO:SOIC-16_3.9x9.9mm_P1.27mm")
     )
     (path "/279c7d5e-a2a5-463c-9a5f-466442a96f2a"
-      (reference "IC2") (unit 5) (value "LM13700N") (footprint "Package_SO:SO-16_5.3x10.2mm_P1.27mm")
+      (reference "IC2") (unit 5) (value "LM13700N") (footprint "Package_SO:SOIC-16_3.9x9.9mm_P1.27mm")
     )
     (path "/47de7e50-8323-450b-8255-418e128952b5"

Commit message: Split up into separate main and io boards, update power silkscreen
Power connector silkscreen was updated to make it more obvious that the
connector is to be mounted on the backside, in the same orientation as
front silk screen.
Parts:
- removed C1, C2, C3, C4: .1uf, ioboard:C050-024X044, symbol ioboard-eagle-import:C-EU050-024X044
- removed C6, C7: 10uf, ioboard:E2,5-5, symbol ioboard-eagle-import:CPOL-USE2.5-5
- removed IC1: TL074P, Package_SO:SO-14_3.9x8.65mm_P1.27mm, symbol ioboard-eagle-import:TL074P
- removed IC2: LM13700N, Package_SO:SOIC-16_3.9x9.9mm_P1.27mm, symbol ioboard-eagle-import:LM13700N
- removed JP3, JP4: PINHD-1X6, ioboard:1X06, symbol ioboard-eagle-import:PINHD-1X6
- removed JP6: PINHD-1X4, ioboard:1X04, symbol ioboard-eagle-import:PINHD-1X4
- removed PWR0: ML10, ioboard:ML10, symbol ioboard-eagle-import:ML10
- removed Q1, Q3: 2N3904, ioboard:TO92, symbol ioboard-eagle-import:2N3904
- removed Q2, Q4: 2N3906, ioboard:TO92, symbol ioboard-eagle-import:2N3906
- removed R1, R2: 100k, Potentiometer_THT:Potentiometer_Bourns_3296W_Vertical, symbol Device:R_Potentiometer_Trim
- removed R10, R30: 47k, ioboard:0204_7, symbol ioboard-eagle-import:R-US_0204/7
- removed R11, R31: 1k, ioboard:0204_7, symbol ioboard-eagle-import:R-US_0204/7
- removed R12, R32: 4.7k, ioboard:0204_7, symbol ioboard-eagle-import:R-US_0204/7
- removed R13, R15, R21, R33, R35, R41: 2k, ioboard:0204_7, symbol ioboard-eagle-import:R-US_0204/7
- removed R14, R22, R23, R28, R34, R42, R43, R8: 100k, ioboard:0204_7, symbol ioboard-eagle-import:R-US_0204/7
- removed R19, R39: 120k, ioboard:0204_7, symbol ioboard-eagle-import:R-US_0204/7
- removed R20, R26, R40, R46: 20k, ioboard:0204_7, symbol ioboard-eagle-import:R-US_0204/7
- removed R24, R44: 470R, ioboard:0204_7, symbol ioboard-eagle-import:R-US_0204/7
- removed R25, R45: 30k, ioboard:0204_7, symbol ioboard-eagle-import:R-US_0204/7
- removed R27, R7: 150R, ioboard:0204_7, symbol ioboard-eagle-import:R-US_0204/7
- removed R29, R9: 470k, ioboard:0204_7, symbol ioboard-eagle-import:R-US_0204/7
- removed R3, R4: 2k, Potentiometer_THT:Potentiometer_Bourns_3296W_Vertical, symbol Device:R_Potentiometer_Trim
- removed R5, R6: 2M, ioboard:0204_7, symbol ioboard-eagle-import:R-US_0204/7
