File: SCM-140-ADSR/mainboard/mainboard.kicad_pcb (KiCad board)
At the start: 2 copper layers, 108 x 48.3 mm, 108 parts, among them IC1 LM4558N, IC2 LM4558N, IC3 LM4558N

Commit message: Also export back silkscreen, and add some missing back silkscreen
Other:
- board text added: "+12V"
- board text added: "-12V"
Changed lines of the file:
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@@
       (net 7 "N$6") (solder_mask_margin 0.1016))
   )
+  (gr_line (start 192.15 95.49) (end 192.15 115.88) (layer "B.SilkS") (width 0.12))
+  (gr_line (start 191.58 103.61) (end 191.58 107.67) (layer "B.SilkS") (width 0.12))
   (gr_line (start 194.2211 100.5586) (end 192.3161 100.5586) (layer "F.SilkS") (width 0.4064))
   (gr_line (start 194.2211 110.7186) (end 192.3161 110.7186) (layer "F.SilkS") (width 0.4064))
@@
   (gr_line (start 202.4761 129.1336) (end 202.4761 80.8736) (layer "Edge.Cuts") (width 0.05))
   (gr_line (start 94.5261 80.8736) (end 94.5261 129.1336) (layer "Edge.Cuts") (width 0.05))
+  (gr_text "+12V" (at 196.69 94.03) (layer "B.SilkS")
+    (effects (font (size 1 1) (thickness 0.15)) (justify mirror))
+  )
+  (gr_text "-12V" (at 197.45 116.93) (layer "B.SilkS")
+    (effects (font (size 1 1) (thickness 0.15)) (justify mirror))
+  )
   (gr_text "-12v" (at 191.6811 113.2586 90) (layer "F.SilkS")
     (effects (font (size 1.308608 1.308608) (thickness 0.113792)) (justify left bottom))
