File: Steiner-VCF/mainboard/mainboard.kicad_pcb (KiCad board)
At the start: 2 copper layers, 38.1 x 99.1 mm, 57 parts, among them IC1 TL074P, T1 BC547C, T2 BC547C

Commit message: Also export back silkscreen, and add some missing back silkscreen
Other:
- board text added: "+12V"
- board text added: "-12V"
Changed lines of the file:
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@@
       (net 40 "Net-(R4-Pad2)") (pinfunction "E") (pintype "passive") (solder_mask_margin 0.1016))
   )
+  (gr_line (start 139.41 152.35) (end 157.62 152.32) (layer "B.SilkS") (width 0.12))
+  (gr_line (start 146.28 152.7) (end 150.66 152.7) (layer "B.SilkS") (width 0.12))
   (gr_circle (center 163.7411 59.2836) (end 166.5351 59.2836) (layer "F.SilkS") (width 0.127) (fill none))
   (gr_line (start 167.5511 55.4736) (end 129.4511 55.4736) (layer "Edge.Cuts") (width 0.05))
@@
   (gr_line (start 129.4511 55.4736) (end 129.4511 154.5336) (layer "Edge.Cuts") (width 0.05))
   (gr_line (start 129.4511 154.5336) (end 167.5511 154.5336) (layer "Edge.Cuts") (width 0.05))
+  (gr_text "-12V" (at 159.73 148.47 90) (layer "B.SilkS")
+    (effects (font (size 1 1) (thickness 0.15)) (justify mirror))
+  )
+  (gr_text "+12V" (at 137.26 148.8 90) (layer "B.SilkS")
+    (effects (font (size 1 1) (thickness 0.15)) (justify mirror))
+  )
   (gr_text "+12v" (at 137.7061 151.3586 90) (layer "F.SilkS")
     (effects (font (size 1.1684 1.1684) (thickness 0.1016)) (justify left bottom))
