File: TH-555-VCO/mainboard/mainboard.kicad_pcb (KiCad board)
At the start: 2 copper layers, 108 x 48.3 mm, 71 parts, among them IC1 555N, IC2 LM13700N, IC3 TL074P, IC4 TL074P, T3 -NPN-TO92-EBC, T4 -PNP-TO92-EBC, T5 -PNP-TO92-EBC

Commit message: Also export back silkscreen, and add some missing back silkscreen
Other:
- board text added: "+12V"
- board text added: "-12V"
Changed lines of the file:
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@@
       (net 44 "Net-(R11-PadS)") (pinfunction "S") (pintype "passive") (solder_mask_margin 0.1016))
   )
+  (gr_line (start 201.32 102.9) (end 201.32 107.09) (layer "B.SilkS") (width 0.12))
+  (gr_line (start 201 95.78) (end 200.97 114.14) (layer "B.SilkS") (width 0.12))
   (gr_line (start 192.3161 115.1636) (end 192.3161 110.0836) (layer "F.SilkS") (width 0.4064))
   (gr_line (start 192.3161 99.9236) (end 192.3161 94.8436) (layer "F.SilkS") (width 0.4064))
@@
   (gr_line (start 202.4761 129.1336) (end 202.4761 80.8736) (layer "Edge.Cuts") (width 0.05))
   (gr_line (start 94.5261 129.1336) (end 202.4761 129.1336) (layer "Edge.Cuts") (width 0.05))
+  (gr_text "+12V" (at 197.5 115.31) (layer "B.SilkS")
+    (effects (font (size 1 1) (thickness 0.15)) (justify mirror))
+  )
+  (gr_text "-12V" (at 197.82 94.88) (layer "B.SilkS")
+    (effects (font (size 1 1) (thickness 0.15)) (justify mirror))
+  )
   (gr_text "SINE ROUND" (at 138.9761 123.4186) (layer "F.SilkS")
     (effects (font (size 1.1684 1.1684) (thickness 0.1016)) (justify left bottom))
