File: AS3340-VCO/ioboard/ioboard.kicad_sch (KiCad schematic)
At the start: 22 parts, among them J1 Conn_02x05_Odd_Even, J10 SINE, J11 SAW, J12 PULSE, J2 Conn_01x03, J3 EXP_FM, J4 CV, J5 PWM, J6 LIN_FM, J7 HARD_SYNC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

Commit message: Finish DuinoRack hardware, final touches on AS3340 VCO
Parts:
- removed J1: Conn_02x05_Odd_Even, Connector_PinHeader_2.54mm:PinHeader_2x05_P2.54mm_Vertical, symbol Connector_Generic:Conn_02x05_Odd_Even
- removed J2: Conn_01x03, Connector_PinHeader_2.54mm:PinHeader_1x03_P2.54mm_Vertical, symbol Connector_Generic:Conn_01x03
- removed TUNE_COARSE1: 100k, Potentiometer_THT:Potentiometer_Alps_RK09K_Single_Vertical, symbol Device:R_Potentiometer
- added C2: 470n, Capacitor_THT:C_Rect_L7.0mm_W3.5mm_P5.00mm, symbol Device:C
- added C3, C4, C5, C6: 100n, Capacitor_SMD:C_0603_1608Metric_Pad1.08x0.95mm_HandSolder, symbol Device:C
- added D1, D2: RB521S30, Diode_SMD:D_SOD-523, symbol Device:D_Schottky
- added D3: LED_Dual_Bidirectional, LED_THT:LED_D3.0mm, symbol Device:LED_Dual_Bidirectional
- added H1: MountingHole, Library:MountingHole_3.2mm_M3_NoCourt, symbol Mechanical:MountingHole
- added J1: Conn_02x06_Odd_Even, Connector_PinHeader_2.54mm:PinHeader_2x06_P2.54mm_Vertical, symbol Connector_Generic:Conn_02x06_Odd_Even
- added J2: Conn_01x04, Connector_PinHeader_2.54mm:PinHeader_1x04_P2.54mm_Vertical, symbol Connector_Generic:Conn_01x04
- added R10, R11, R5, R6, R7, R8, R9: 10k 0.1%, Resistor_SMD:R_0603_1608Metric_Pad0.98x0.95mm_HandSolder, symbol Device:R
- added R12: 3.3k, Resistor_SMD:R_0603_1608Metric_Pad0.98x0.95mm_HandSolder, symbol Device:R
- added R13: 3.9k, Resistor_SMD:R_0603_1608Metric_Pad0.98x0.95mm_HandSolder, symbol Device:R
- added SW1: OCT, Library:Rotary-Switch-8-ALPS-SRBV, symbol TuringFront-eagle-import:ALPS-SRBV
- added SW2: SW_LFO, Library:SW_Toggle_Blue_wSlots, symbol Switch:SW_SPDT
- added U1: TL072, Package_SO:SOIC-8_3.9x4.9mm_P1.27mm, symbol Amplifier_Operational:TL072
- R1: value 3.3M -> 100k 0.1%
- R2, R3, R4: value 100k -> 100k 0.1%
Connections:
- net +12V: now also C3.1, J2.1 (Pin_1), U1.8 (V+); no longer TUNE_FINE1.3
- net -12V: now also C4.2, J2.3 (Pin_3), U1.4 (V-)
- net GND: now also C2.2, C3.2, C4.1, C5.2, C6.2, D3.1 (KA), J2.2 (Pin_2), R11.2, SW1.A (1)
- net HARD_SYNC: now also J1.9 (Pin_9)
- net LIN_FM: now also J1.3 (Pin_3)
- net PULSE: now also J1.10 (Pin_10)
- net PWM: now also J1.5 (Pin_5)
- net SAW: now also J1.8 (Pin_8)
- net SINE: now also J1.6 (Pin_6)
- net SOFT_SYNC: now also J1.2 (Pin_2)
- net TRIANGLE: now also D1.2 (A), D2.1 (K), J1.4 (Pin_4)
- net VFCI: now also J1.1 (Pin_1)
- net WIDTH: now also J1.7 (Pin_7)
- net at TUNE_FINE1.2: now also U1.5 (+); no longer R1.1
- net at R2.1: now also U1.1, U1.2 (-)
- new net: R10.1, R9.2, SW1.C (3)
- new net: R10.2, R11.1, SW1.B (2)
- new net: R1.1, U1.6 (-), U1.7
- new net: D1.1 (K), R12.1
- new net: R5.2, R6.1, SW1.G (7)
- new net: D3.2 (AK), R12.2, R13.2
- new net: SW1.COM (A), SW1.COM2 (A), U1.3 (+)
- new net: R8.2, R9.1, SW1.D (4)
- new net: R7.2, R8.1, SW1.E (5)
- new net: R6.2, R7.1, SW1.F (6)
- new net: C6.1, D2.2 (A), R13.1
- new net: C2.1, SW2.1 (A)
- new net +7.000V: J2.4 (Pin_4), R5.1, SW1.H (8)
- new net 1V: C5.1, J1.11 (Pin_11), TUNE_FINE1.3
- new net CAP: J1.12 (Pin_12), SW2.2 (B)
- no-connect marks 4 -> 5
Other:
- moved on the sheet: R1, R2, TUNE_FINE1
