File: AS3340-VCO/ioboard/ioboard.kicad_pcb (KiCad board)
At the start: 2 copper layers, 34.9 x 108 mm, 24 parts, among them J1 Conn_02x05_Odd_Even, J10 SINE, J11 SAW, J12 PULSE, J2 Conn_01x03, J3 EXP_FM, J4 CV, J5 PWM, J6 LIN_FM, J7 HARD_SYNC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

Commit message: Finish DuinoRack hardware, final touches on AS3340 VCO
Parts:
- removed REF** (x2): MountingHole_3.2mm_M3_NoCourt, Library:MountingHole_3.2mm_M3_NoCourt
- removed TUNE_COARSE1: 100k, Potentiometer_THT:Potentiometer_Alps_RK09K_Single_Vertical
- added C2: 470n, Capacitor_THT:C_Rect_L7.0mm_W3.5mm_P5.00mm, F.Cu at (147.2, 73.0)
- added C3: 100n, Capacitor_SMD:C_0603_1608Metric_Pad1.08x0.95mm_HandSolder, B.Cu at (155.3, 78.2)
- added C4: 100n, Capacitor_SMD:C_0603_1608Metric_Pad1.08x0.95mm_HandSolder, B.Cu at (163.5, 72.1)
- added C5: 100n, Capacitor_SMD:C_0603_1608Metric_Pad1.08x0.95mm_HandSolder, B.Cu at (164.4, 54.0)
- added C6: 100n, Capacitor_SMD:C_0603_1608Metric_Pad1.08x0.95mm_HandSolder, B.Cu at (134.7, 130.3)
- added D1: RB521S30, Diode_SMD:D_SOD-523, B.Cu at (139.3, 127.0)
- added D2: RB521S30, Diode_SMD:D_SOD-523, B.Cu at (133.1, 128.1)
- added D3: LED_Dual_Bidirectional, LED_THT:LED_D3.0mm, F.Cu at (136.8, 131.3)
- added H1: MountingHole, Library:MountingHole_3.2mm_M3_NoCourt, F.Cu at (162.2, 116.2)
- added R10: 10k 0.1%, Resistor_SMD:R_0603_1608Metric_Pad0.98x0.95mm_HandSolder, B.Cu at (153.0, 67.4)
- added R11: 10k 0.1%, Resistor_SMD:R_0603_1608Metric_Pad0.98x0.95mm_HandSolder, B.Cu at (156.3, 67.4)
- added R12: 3.3k, Resistor_SMD:R_0603_1608Metric_Pad0.98x0.95mm_HandSolder, B.Cu at (141.5, 128.0)
- added R13: 3.9k, Resistor_SMD:R_0603_1608Metric_Pad0.98x0.95mm_HandSolder, B.Cu at (135.6, 127.6)
- added R5: 10k 0.1%, Resistor_SMD:R_0603_1608Metric_Pad0.98x0.95mm_HandSolder, B.Cu at (156.7, 53.9)
- added R6: 10k 0.1%, Resistor_SMD:R_0603_1608Metric_Pad0.98x0.95mm_HandSolder, B.Cu at (153.2, 53.9)
- added R7: 10k 0.1%, Resistor_SMD:R_0603_1608Metric_Pad0.98x0.95mm_HandSolder, B.Cu at (149.8, 53.8)
- added R8: 10k 0.1%, Resistor_SMD:R_0603_1608Metric_Pad0.98x0.95mm_HandSolder, B.Cu at (148.5, 64.8)
- added R9: 10k 0.1%, Resistor_SMD:R_0603_1608Metric_Pad0.98x0.95mm_HandSolder, B.Cu at (149.4, 67.4)
- added SW1: OCT, Library:Rotary-Switch-8-ALPS-SRBV, F.Cu at (154.0, 60.7)
- added SW2: SW_LFO, Library:SW_Toggle_Blue_wSlots, F.Cu at (138.5, 70.4)
- added U1: TL072, Package_SO:SOIC-8_3.9x4.9mm_P1.27mm, B.Cu at (159.8, 75.6)
- J1: value Conn_02x05_Odd_Even -> Conn_02x06_Odd_Even; footprint Connector_PinHeader_2.54mm:PinHeader_2x05_P2.54mm_Vertical -> Connector_PinHeader_2.54mm:PinHeader_2x06_P2.54mm_Vertical
- J2: value Conn_01x03 -> Conn_01x04; footprint Connector_PinHeader_2.54mm:PinHeader_1x03_P2.54mm_Vertical -> Connector_PinHeader_2.54mm:PinHeader_1x04_P2.54mm_Vertical
- R1: value 3.3M -> 100k 0.1%
- R2, R3, R4: value 100k -> 100k 0.1%
- moved J9 10.6 mm to (144.5, 123.5), turned to -90 degrees
- moved J12 10.5 mm to (151.7, 123.5), turned to 90 degrees
- moved J8 8.77 mm to (158.5, 113.2), turned to -90 degrees
- moved C1 5.75 mm to (141.2, 105.2), turned to 180 degrees
- moved RV_LIN_FM_AT1 5.54 mm to (134.1, 88.5)
- moved WIDTH1 5.54 mm to (157.2, 88.5)
- moved RV_EXP_FM_AT1 5.54 mm to (145.6, 92.5)
- moved J3 4.96 mm to (148.1, 95.1)
- moved J5 4.96 mm to (159.7, 91.2)
- moved J6 4.96 mm to (136.6, 91.2)
- moved J7 4.90 mm to (144.3, 113.2)
- moved J1 1.00 mm to (151.3, 42.4)
- moved R1 1.00 mm to (151.9, 45.9)
- moved R2 1.00 mm to (150.3, 45.9)
- moved R3 1.00 mm to (148.6, 43.1)
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Connections:
- TUNE_FINE1 pad 2: Net-(R1-Pad1) -> Net-(TUNE_FINE1-Pad2)
- TUNE_FINE1 pad 3: +12V -> /1V
Routing:
- net /+7.000V: track 0.00 -> 88.3 mm
- net GND: track 0.00 -> 76.7 mm, vias 0 -> 4
- net Net-(TUNE_FINE1-Pad2): track 0.00 -> 57.1 mm, vias 0 -> 1
- net /CAP: track 0.00 -> 54.7 mm
- net +12V: track 112.0 -> 59.2 mm, vias 0 -> 1
- net /1V: track 0.00 -> 48.9 mm
- net Net-(R2-Pad1): track 16.5 -> 38.8 mm
- net Net-(SW1-PadCOM): track 0.00 -> 22.1 mm
- net Net-(R1-Pad1): track 24.8 -> 45.2 mm, vias 0 -> 3
- net -12V: track 52.2 -> 68.9 mm, vias 1 -> 2
- net Net-(C2-Pad1): track 0.00 -> 14.8 mm
- net Net-(R7-Pad2): track 0.00 -> 12.5 mm
- net /HARD_SYNC: track 90.3 -> 101.8 mm
- net /TRIANGLE: track 95.8 -> 107.4 mm, vias 0 -> 1
- net /SOFT_SYNC: track 75.8 -> 86.7 mm
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Other:
- board text added: "100k 0.1%"
- board text added: "K"

Commit message: Saving latest changes
Parts:
- J10, J11, J12, J3, J4, J5, J6, J7, J8, J9: footprint Connector_Audio:Jack_3.5mm_QingPu_WQP-PJ398SM_Vertical_CircularHoles -> Library:Jack_3.5mm_QingPu_WQP-PJ398SM_Vertical_CircularHoles_Hole
