File: DuinoRack/mainboard/mainboard.kicad_sch (KiCad schematic)
At the start: 122 parts, among them J2 SER, J3 Conn_02x08_Odd_Even, J4 Conn_02x05_Odd_Even, J5 Conn_MIDI, J6 Conn_02x03_Odd_Even, U1 MCP4822, U2 ATmega328P-P, U3 TL074, U4 TL431DBZ, U5 MCP6004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

Commit message: Saving latest changes
Parts:
- added D2: 1N4148WS, Diode_SMD:D_SOD-323_HandSoldering, symbol Device:D
Connections:
- net +5V: now also D2.1 (K); no longer J2.3 (Pin_3)
- new net: D2.2 (A), J2.3 (Pin_3)
Changed lines of the file:
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@@
     (pin "1")
   )
+  (symbol (lib_id "Device:D") (at 153.67 39.37 0) (mirror x) (unit 1)
+    (in_bom yes) (on_board yes) (fields_autoplaced)
+    (property "Reference" "D2" (id 0) (at 153.67 33.02 0))
+    (property "Value" "1N4148WS" (id 1) (at 153.67 35.56 0))
+    (property "Footprint" "Diode_SMD:D_SOD-323_HandSoldering" (id 2) (at 153.67 39.37 0)
+      (effects (font (size 1.27 1.27)) hide)
+    )
+    (property "Datasheet" "~" (id 3) (at 153.67 39.37 0)
+      (effects (font (size 1.27 1.27)) hide)
+    )
+    (pin "1")
+    (pin "2")
+  )
   (symbol (lib_id "power:GND") (at 123.19 172.72 0) (unit 1)
     (in_bom yes) (on_board yes) (fields_autoplaced)
@@
     (pin "2")
   )
-  (symbol (lib_id "power:+5V") (at 157.48 39.37 90) (unit 1)
+  (symbol (lib_id "power:+5V") (at 149.86 39.37 90) (unit 1)
     (in_bom yes) (on_board yes) (fields_autoplaced)
-    (property "Reference" "#PWR05" (id 0) (at 161.29 39.37 0)
+    (property "Reference" "#PWR05" (id 0) (at 153.67 39.37 0)
       (effects (font (size 1.27 1.27)) hide)
     )
-    (property "Value" "+5V" (id 1) (at 153.67 39.3699 90)
+    (property "Value" "+5V" (id 1) (at 146.05 39.3699 90)
       (effects (font (size 1.27 1.27)) (justify left))
     )
-    (property "Footprint" "" (id 2) (at 157.48 39.37 0)
+    (property "Footprint" "" (id 2) (at 149.86 39.37 0)
       (effects (font (size 1.27 1.27)) hide)
     )
-    (property "Datasheet" "" (id 3) (at 157.48 39.37 0)
+    (property "Datasheet" "" (id 3) (at 149.86 39.37 0)
       (effects (font (size 1.27 1.27)) hide)
     )
@@
       (reference "D1") (unit 1) (value "5.1V") (footprint "Diode_THT:D_DO-35_SOD27_P2.54mm_Vertical_AnodeUp")
     )
+    (path "/0f3c536f-0cd8-4d20-a612-26b98ae21b0c"
+      (reference "D2") (unit 1) (value "1N4148WS") (footprint "Diode_SMD:D_SOD-323_HandSoldering")
+    )
     (path "/600de48d-5417-4381-87fe-6b6822ea96e5"
