File: PT2399-Delay/faceplate/faceplate.kicad_pcb (KiCad board)
At the start: 2 copper layers, 20.1 x 128.5 mm, 8 parts

Commit message: Small updates for delay while ordering first prototype
Other:
- board text added: "JLCJLCJLCJLC"
Changed lines of the file:
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@@
 		(layer "Edge.Cuts")
+	)
+	(gr_text "JLCJLCJLCJLC"
+		(at 98.45 158.3 0)
+		(layer "B.SilkS")
+		(effects
+			(font
+				(size 0.8 0.8)
+				(thickness 0.1)
+			)
+			(justify left bottom mirror)
+		)
 	)
 	(zone
