File: PT2399-Delay/mainboard/mainboard.kicad_pcb (KiCad board)
At the start: 2 copper layers, 19 x 107.9 mm, 72 parts, among them J1 Conn_02x05_Odd_Even, J2 Conn_02x05_Odd_Even, Q1 3416, Q3 MMBT3904, U1 PT2399, U2 TL074, U3 TL074, U5 LM7805_TO220

Commit message: Adjust layout so components can be folded over
Parts:
- moved C17 10.3 mm to (91.4, 126.1), turned to -90 degrees
- moved U5 6.44 mm to (90.7, 121.1)
- moved C18 1.38 mm to (91.4, 132.2), turned to 90 degrees
- moved D1 0.43 mm to (87.7, 132.6)
Routing:
- net GND: track 43.8 -> 93.2 mm, vias 6 -> 12
- net +5V: track 77.5 -> 86.1 mm
- net +12V: track 108.6 -> 106.1 mm
- net -12V: track 124.7 -> 126.9 mm, vias 4 -> 3
Other:
- board text added: "7805"

Commit message: Small updates for delay while ordering first prototype
Other:
- board text added: "+12V"
- board text added: "-12V"
Changed lines of the file:
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@@
 		(tags "CP Radial series Radial pin pitch 1.50mm  diameter 4mm Electrolytic Capacitor")
 		(property "Reference" "C18"
-			(at -2.19 1.14 360)
+			(at -2.19 1.14 0)
 			(layer "F.SilkS")
 			(effects
@@
 		)
 		(property "Value" "10u"
-			(at -3.33 1.4 360)
+			(at -3.33 1.4 0)
 			(layer "F.SilkS")
 			(effects
@@
 		)
 		(fp_text user "${REFERENCE}"
-			(at 2.54 -4.27 360)
+			(at 2.54 -4.27 0)
 			(layer "F.Fab")
 			(effects
@@
 		(tags "Through hole pin header THT 2x05 2.54mm double row")
 		(property "Reference" "J1"
-			(at 1.27 2.33 90)
+			(at -0.73 2.43 90)
 			(layer "B.SilkS")
 			(effects
@@
 		(layer "Edge.Cuts")
 	)
+	(gr_text "-12V"
+		(at 77.62 139.08 90)
+		(layer "B.SilkS")
+		(effects
+			(font
+				(size 0.8 0.8)
+				(thickness 0.1)
+			)
+			(justify left bottom mirror)
+		)
+	)
+	(gr_text "+12V"
+		(at 92.81 138.53 90)
+		(layer "B.SilkS")
+		(effects
+			(font
+				(size 0.8 0.8)
+				(thickness 0.1)
+			)
+			(justify left bottom mirror)
+		)
+	)
 	(gr_text "7805"
