File: DualMixer/ioboard/ioboard.kicad_sch (KiCad schematic)
At the start: 22 parts, among them J1 IN_A1, J10 IN_B4, J11 OUTB, J13 Conn_01x03_Male, J2 IN_A2, J3 IN_A3, J4 OUTA, J5 Conn_02x07_Odd_Even, J6 IN_A4, J7 IN_B1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

Commit message: Apply fixes for DualMixer rev1 module
Connections:
- net GND: now also RV_A1.1, RV_A2.1, RV_A3.1, RV_A4.1, RV_B1.1, RV_B2.1, RV_B3.1, RV_B4.1; no longer RV_A1.3, RV_A2.3, RV_A3.3, RV_A4.3, RV_B1.3, RV_B2.3, RV_B3.3, RV_B4.3
- net at J9.T: now also RV_B3.3; no longer RV_B3.1
- net at J7.T: now also RV_B1.3; no longer RV_B1.1
- net at J3.T: now also RV_A3.3; no longer RV_A3.1
- net at J6.T: now also RV_A4.3; no longer RV_A4.1
- net at J8.T: now also RV_B2.3; no longer RV_B2.1
- net at J1.T: now also RV_A1.3; no longer RV_A1.1
- net at J2.T: now also RV_A2.3; no longer RV_A2.1
- net at J10.T: now also RV_B4.3; no longer RV_B4.1
